File: inspireFly-flightController/inspireFly-flightController.kicad_pcb (KiCad board)
At the start: 4 copper layers, 95.6 x 80 mm, 31 parts, among them J1 FTSH-107-01-L-DV-K-A, SW1 SW_Push, SW3 SW_Push, U1 STM32U595VJT6, U2 BNO086, Y1 ABS07-32.768KHZ-T

Commit message: fixed up schematic and pcb
Parts:
- added C17: 22pF, Capacitor_SMD:C_0402_1005Metric_Pad0.74x0.62mm_HandSolder, F.Cu at (99.1, 86.0)
- added C18: 22pF, Capacitor_SMD:C_0402_1005Metric_Pad0.74x0.62mm_HandSolder, F.Cu at (104.2, 86.0)
- added Y2: ABS07-32.768KHZ-T, flightController:XTAL_ABS07-32.768KHZ-T, F.Cu at (101.7, 85.9)
- J1: footprint inspirefly:SAMTEC_FTSH-107-01-L-DV-K-A -> flightController:SAMTEC_FTSH-107-01-L-DV-K-A
- R10: footprint Resistor_SMD:R_0402_1005Metric -> Resistor_SMD:R_0402_1005Metric_Pad0.72x0.64mm_HandSolder
- Y1: footprint inspirefly:XTAL_ABS07-32.768KHZ-T -> flightController:XTAL_ABS07-32.768KHZ-T
- moved C15 0.30 mm to (98.5, 94.6)
Connections:
- U1 pad 39: IMU_PSO/WAKE_GPIO -> unconnected-(U1-PE8-Pad39)
- U2 pad 26: GND -> Net-(U2-XOUT32/CLKSEL1)
- U2 pad 27: unconnected-(U2-XIN32-Pad27) -> Net-(U2-XIN32)
Routing:
- net Net-(U2-XOUT32/CLKSEL1): track 0.00 -> 8.37 mm
- net IMU_PSO/WAKE_GPIO: track 41.9 -> 37.5 mm
- net Net-(U2-XIN32): track 0.00 -> 4.39 mm
