File: inspireFly-flightController/inspireFly-flightController.kicad_pcb (KiCad board)
At the start: 4 copper layers, 95.6 x 80 mm, 64 parts, among them J1 FTSH-107-01-L-DV-K-A, SW1 SW_Push, SW3 SW_Push, U1 STM32U595VJT6, U2 BNO086, U3 RV-8803-C7, U4 LM66100DCK, U5 TPS2117, U6 RV-8803-C7, Y1 ABS07-32.768KHZ-T, Y2 ABS07-32.768KHZ-T

Commit message: Interfaced 1GB flash storage IC onto PCB, updated footprints
Parts:
- added C21: 1.5F, inspirefly:SUPERCAP_KR-5R5H155-R, F.Cu at (64.5, 141.8)
- added C28: 1uF, Capacitor_SMD:C_0402_1005Metric_Pad0.74x0.62mm_HandSolder, F.Cu at (111.9, 105.3)
- added C31: 1.5F, inspirefly:SUPERCAP_KR-5R5H155-R, F.Cu at (64.5, 162.1)
- added C32: 100nF, Capacitor_SMD:C_0402_1005Metric_Pad0.74x0.62mm_HandSolder, F.Cu at (114.4, 105.3)
- added C33: 100nF, Capacitor_SMD:C_0402_1005Metric_Pad0.74x0.62mm_HandSolder, F.Cu at (139.9, 106.2)
- added R18: 4.7k, Resistor_SMD:R_0402_1005Metric_Pad0.72x0.64mm_HandSolder, F.Cu at (78.4, 148.0)
- added R38: 10K, Resistor_SMD:R_0402_1005Metric_Pad0.72x0.64mm_HandSolder, F.Cu at (114.4, 108.8)
- added R39: 4.7K, Resistor_SMD:R_0402_1005Metric_Pad0.72x0.64mm_HandSolder, F.Cu at (113.9, 99.7)
- added R40: 10K, Resistor_SMD:R_0402_1005Metric_Pad0.72x0.64mm_HandSolder, F.Cu at (112.9, 102.0)
- added R7: 4.7k, Resistor_SMD:R_0402_1005Metric_Pad0.72x0.64mm_HandSolder, F.Cu at (78.4, 146.0)
- added TP2: VCAP_A2, TestPoint:TestPoint_Pad_D1.5mm, F.Cu at (81.8, 146.8)
- added TP8: VCAP_B2, TestPoint:TestPoint_Pad_D1.5mm, F.Cu at (81.8, 150.3)
- added U7: MX60LF8G28AD-TI, Flash_Storage:TSOPI48_MAC, F.Cu at (127.0, 105.0)
- TP1: value VCAP_A1 -> VACP_A1
Connections:
- U1 pad 35: unconnected-(U1-PB0-Pad35) -> WP#
- U1 pad 38: unconnected-(U1-PE7-Pad38) -> I/O4
- U1 pad 39: unconnected-(U1-PE8-Pad39) -> I/O5
- U1 pad 40: unconnected-(U1-PE9-Pad40) -> I/O6
- U1 pad 41: unconnected-(U1-PE10-Pad41) -> I/O7
- U1 pad 58: unconnected-(U1-PD11-Pad58) -> CLE
- U1 pad 59: unconnected-(U1-PD12-Pad59) -> ALE
- U1 pad 61: unconnected-(U1-PD14-Pad61) -> I/O0
- U1 pad 62: unconnected-(U1-PD15-Pad62) -> I/O1
- U1 pad 81: unconnected-(U1-PD0-Pad81) -> I/O2
- U1 pad 82: unconnected-(U1-PD1-Pad82) -> I/O3
- U1 pad 85: unconnected-(U1-PD4-Pad85) -> RE#
- U1 pad 86: unconnected-(U1-PD5-Pad86) -> WE#
- U1 pad 87: unconnected-(U1-PD6-Pad87) -> R/B#
- U1 pad 88: unconnected-(U1-PD7-Pad88) -> CE#
Routing:
- net WE#: track 0.00 -> 59.9 mm, vias 0 -> 4
- net ALE: track 0.00 -> 47.4 mm, vias 0 -> 4
- net CE#: track 0.00 -> 46.5 mm, vias 0 -> 6
- net I/O2: track 0.00 -> 45.8 mm, vias 0 -> 2
- net I/O3: track 0.00 -> 45.8 mm, vias 0 -> 2
- net I/O1: track 0.00 -> 45.7 mm, vias 0 -> 2
- net I/O6: track 0.00 -> 45.7 mm, vias 0 -> 2
- net I/O0: track 0.00 -> 45.7 mm, vias 0 -> 2
- net I/O7: track 0.00 -> 45.6 mm, vias 0 -> 2
- net I/O5: track 0.00 -> 45.6 mm, vias 0 -> 2
- net I/O4: track 0.00 -> 45.5 mm, vias 0 -> 2
- net R/B#: track 0.00 -> 37.3 mm, vias 0 -> 2
- net RE#: track 0.00 -> 36.8 mm, vias 0 -> 4
- net CLE: track 0.00 -> 35.6 mm, vias 0 -> 2
- net WP#: track 0.00 -> 27.3 mm, vias 0 -> 2
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