File: inspireFly-flightController/inspireFly-flightController.kicad_sch (KiCad schematic)
At the start: 31 parts, among them J1 FTSH-107-01-L-DV-K-A, SW1 SW_Push, SW3 SW_Push, U1 STM32U595VJT6, U2 BNO086, Y1 ABS07-32.768KHZ-T

Commit message: fixed up schematic and pcb
Parts:
- added C17, C18: 22pF, Capacitor_SMD:C_0402_1005Metric_Pad0.74x0.62mm_HandSolder, symbol Device:C_Small
- added Y2: ABS07-32.768KHZ-T, flightController:XTAL_ABS07-32.768KHZ-T, symbol flightController:ABS07-32.768KHZ-T
- J1: footprint inspirefly:SAMTEC_FTSH-107-01-L-DV-K-A -> flightController:SAMTEC_FTSH-107-01-L-DV-K-A
- R10: footprint Resistor_SMD:R_0402_1005Metric -> Resistor_SMD:R_0402_1005Metric_Pad0.72x0.64mm_HandSolder
- Y1: footprint inspirefly:XTAL_ABS07-32.768KHZ-T -> flightController:XTAL_ABS07-32.768KHZ-T
Connections:
- net GND: now also C17.1, C18.1; no longer U2.26 (XOUT32/CLKSEL1)
- net IMU_PSO/WAKE_GPIO: no longer U1.39 (PE8)
- net at U2.27 (XIN32): now also C17.2, Y2.1
- new net: C18.2, U2.26 (XOUT32/CLKSEL1), Y2.2
- no-connect marks 15 -> 14
