File: inspireFly-flightController/inspireFly-flightController.kicad_sch (KiCad schematic)
At the start: 34 parts, among them J1 FTSH-107-01-L-DV-K-A, SW1 SW_Push, SW3 SW_Push, U1 STM32U595VJT6, U2 BNO086, Y1 ABS07-32.768KHZ-T, Y2 ABS07-32.768KHZ-T

Commit message: added RTC, backup power supply, ideal diode, and switch IC
Parts:
- added C19, C29: 10nF, Capacitor_SMD:C_0402_1005Metric_Pad0.74x0.62mm_HandSolder, symbol Device:C_Small
- added C20, C21, C30, C31: 1.5F, flightController:SUPERCAP_KR-5R5H155-R, symbol Device:C_Polarized
- added C23, C24, C25, C27: 1uF, Capacitor_SMD:C_0402_1005Metric_Pad0.74x0.62mm_HandSolder, symbol Device:C_Small
- added R11, R12, R8: 100k, Resistor_SMD:R_0402_1005Metric_Pad0.72x0.64mm_HandSolder, symbol Device:R_US
- added R13, R14, R15, R16, R2, R3, R4, R5: 10k, Resistor_SMD:R_0402_1005Metric_Pad0.72x0.64mm_HandSolder, symbol Device:R_US
- added R17, R18, R6, R7: 4.7k, Resistor_SMD:R_0402_1005Metric_Pad0.72x0.64mm_HandSolder, symbol Device:R_US
- added R9: 150k, Resistor_SMD:R_0402_1005Metric_Pad0.72x0.64mm_HandSolder, symbol Device:R_US
- added TP1, TP2, TP3, TP4, TP5, TP6, TP7, TP8: TestPoint, TestPoint:TestPoint_Pad_D1.5mm, symbol Connector:TestPoint
- added U3, U6: RV-8803-C7, flightController:RTC_RV-8803-C7, symbol flightController:RV-8803-C7
- added U4: LM66100DCK, Package_TO_SOT_SMD:SOT-363_SC-70-6, symbol Power_Management:LM66100DCK
- added U5: TPS2117, flightController:PWRMUX_TPS2117-DRL, symbol flightController:TPS2117
Connections:
- net +3.3V: now also C23.2, C25.1, R12.1, R13.2, R14.2, R15.2, R3.2, R4.2, R5.2, R8.2, R9.1, U4.1 (VIN), U5.3 (VIN1), U5.5 (MODE)
- net GND: now also C19.1, C20.2, C21.2, C23.1, C24.2, C25.2, C27.2, C29.1, C30.2, C31.2, R11.1, U3.4 (CLKOE), U3.5 (VSS), U4.2 (GND), U5.1 (GND), U5.6 (VIN2), U6.4 (CLKOE), U6.5 (VSS)
- net RTC_B_INT: now reaches U1.23 (PA0)
- net RTC_B_INT: now also R15.1, U6.6 (~{INT})
- net RTC_A_INT: now reaches U1.24 (PA1)
- net RTC_A_INT: now also R5.1, U3.6 (~{INT})
- net RTC_B_SCL: now reaches U1.52 (PB13)
- net RTC_B_SCL: now also R13.1, U6.8 (SCL)
- net RTC_B_SDA: now reaches U1.53 (PB14)
- net RTC_B_SDA: now also R14.1, U6.1 (SDA)
- net RTC_A_PWR_ST: now reaches U1.83 (PD2)
- net RTC_A_PWR_ST: now also R8.1, TP4.1, U4.5 (ST)
- net RTC_B_PWR_ST: now reaches U1.84 (PD3)
- net RTC_B_PWR_ST: now also R12.2, TP5.1, U5.8 (ST)
- net RTC_A_SCL: now reaches U1.92 (PB6)
- net RTC_A_SCL: now also R3.1, U3.8 (SCL)
- net RTC_A_SDA: now reaches U1.93 (PB7)
- net RTC_A_SDA: now also R4.1, U3.1 (SDA)
- new net: R11.2, R9.2, U5.4 (PR1)
- new net: R16.2, U6.7 (EVI)
- new net: R2.2, U3.7 (EVI)
- new net VCAP_A1: C20.1, R6.1, TP2.1
- new net VCAP_A2: C21.1, R7.1, TP1.1
- new net VCAP_B1: C30.1, R17.1, TP7.1
- new net VCAP_B2: C31.1, R18.1, TP8.1
- new net VRTC_A: C19.2, C24.1, R2.1, R6.2, R7.2, TP3.1, U3.3 (VDD), U4.3 (~{CE}), U4.6 (VOUT)
- new net VRTC_B: C27.1, C29.2, R16.1, R17.2, R18.2, TP6.1, U5.2 (VOUT), U5.7 (VOUT), U6.3 (VDD)
- no-connect marks 14 -> 16
Other:
- note added: "IMU"
- note added: "Ideal diode"
- note added: "RTC_A"
- note added: "RTC_B"
- note added: "ST-LINK"
- note added: "Switching IC"
- note added: "supercaps_A"
- note added: "supercaps_B"
- moved on the sheet: C7

Commit message: fixed issues, added names to testpoints
Parts:
- removed R16, R2: 10k, Resistor_SMD:R_0402_1005Metric_Pad0.72x0.64mm_HandSolder, symbol Device:R_US
- C20, C21, C30, C31: footprint flightController:SUPERCAP_KR-5R5H155-R -> inspirefly:SUPERCAP_KR-5R5H155-R
- J1: footprint flightController:SAMTEC_FTSH-107-01-L-DV-K-A -> inspirefly:SAMTEC_FTSH-107-01-L-DV-K-A
- TP1: renamed from TP2; value TestPoint -> VACP_A1
- TP2: renamed from TP1; value TestPoint -> VCAP_A2
- TP3: value TestPoint -> VRTC_A
- TP4: value TestPoint -> RTC_A_ST
- TP5: value TestPoint -> RTC_B_ST
- TP6: value TestPoint -> VRTC_B
- TP7: value TestPoint -> VCAP_B1
- TP8: value TestPoint -> VCAP_B2
- U3, U6: footprint flightController:RTC_RV-8803-C7 -> inspirefly:RTC_RV-8803-C7
- U5: footprint flightController:PWRMUX_TPS2117-DRL -> inspirefly:PWRMUX_TPS2117-DRL
- Y1, Y2: footprint flightController:XTAL_ABS07-32.768KHZ-T -> inspirefly:XTAL_ABS07-32.768KHZ-T
Connections:
- net GND: now also U3.7 (EVI), U6.7 (EVI)
Other:
- moved on the sheet: C20, C21, R6, R7, TP1, TP2

Commit message: Interfaced 1GB flash storage IC onto schematic
Parts:
- added C28: 1uF, Capacitor_SMD:C_0402_1005Metric_Pad0.74x0.62mm_HandSolder, symbol Device:C
- added C32: 100nF, Capacitor_SMD:C_0402_1005Metric_Pad0.74x0.62mm_HandSolder, symbol Device:C
- added R38: 10K, Resistor_SMD:R_0402_1005Metric_Pad0.72x0.64mm_HandSolder, symbol Device:R_US
- added U7: MX60LF8G28AD-TI, TSOPI48_MAC, symbol 2026-10-05_16-42-47:MX60LF8G28AD-TI
Connections:
- net +3.3V: now also C28.1, C32.1, R38.2, U7.12 (VCC), U7.34 (VCC), U7.37 (VCC), U7.39 (VCC)
- net GND: now also C28.2, C32.2, U7.13 (VSS), U7.25 (VSS), U7.36 (VSS), U7.48 (VSS)
- net WP#: now reaches U1.35 (PB0)
- net WP#: now also R38.1, U7.19 (WP#)
- net I/O4: now reaches U1.38 (PE7)
- net I/O4: now also U7.41 (I/O4)
- net I/O5: now reaches U1.39 (PE8)
- net I/O5: now also U7.42 (I/O5)
- net I/O6: now reaches U1.40 (PE9)
- net I/O6: now also U7.43 (I/O6)
- net I/O7: now reaches U1.41 (PE10)
- net I/O7: now also U7.44 (I/O7)
- net CLE: now reaches U1.58 (PD11)
- net CLE: now also U7.16 (CLE)
- net ALE: now reaches U1.59 (PD12)
- net ALE: now also U7.17 (ALE)
- net I/O0: now reaches U1.61 (PD14)
- net I/O0: now also U7.29 (I/O0)
- net I/O1: now reaches U1.62 (PD15)
- net I/O1: now also U7.30 (I/O1)
- net I/O2: now reaches U1.81 (PD0)
- net I/O2: now also U7.31 (I/O2)
- net I/O3: now reaches U1.82 (PD1)
- net I/O3: now also U7.32 (I/O3)
- net RE#: now reaches U1.85 (PD4)
- net RE#: now also U7.8 (RE#)
- net WE#: now reaches U1.86 (PD5)
- net WE#: now also U7.18 (WE#)
- net R/B#: now reaches U1.87 (PD6)
- net R/B#: now also U7.7 (R/B#)
- net CE#: now reaches U1.88 (PD7)
- net CE#: now also U7.9 (CE#)
